File: therm-coast.brd (EAGLE design)
At the start: 33 x 33 mm, 20 parts, among them U1 ATTINY85-20SU

Commit message: 1.2
Parts:
- moved R6 2.01 mm to (6.99, 23.5)
Routing:
- net RESET: track 12.8 -> 15.0 mm
- net VCC: track 89.4 -> 87.8 mm, vias 4 -> 3
- net LED_DATA: vias 0 -> 2
Changed lines of the file:
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@@
 </class>
 </classes>
-<designrules name="oshpark-2-layer">
-<description language="de">&lt;b&gt;EAGLE Design Rules&lt;/b&gt;
+<designrules name="oshpark-2layer">
+<description language="en">&lt;b&gt;OSH Park Design Rules&lt;/b&gt;
 &lt;p&gt;
-Die Standard-Design-Rules sind so gewählt, dass sie für
-die meisten Anwendungen passen. Sollte ihre Platine
-besondere Anforderungen haben, treffen Sie die erforderlichen
-Einstellungen hier und speichern die Design Rules unter
-einem neuen Namen ab.</description>
-<description language="en">&lt;b&gt;Laen's PCB Order Design Rules&lt;/b&gt;
+Please make sure your boards conform to these design rules.
+&lt;/p&gt;
 &lt;p&gt;
-Please make sure your boards conform to these design rules.</description>
+Note, that not all DRC settings must be set by the manufacturer. Several can be adjusted for the design, including those listed on our docs page here.
+&lt;a href=&quot;http://docs.oshpark.com/design-tools/eagle/design-rules-files/&quot;&gt;Adjustable Settings&lt;/a&gt;
+&lt;/p&gt;</description>
 <param name="layerSetup" value="(1*16)"/>
-<param name="mtCopper" value="0.0356mm 0.0356mm 0.0356mm 0.0356mm 0.0356mm 0.0356mm 0.0356mm 0.0356mm 0.0356mm 0.0356mm 0.0356mm 0.0356mm 0.0356mm 0.0356mm 0.0356mm 0.0356mm"/>
-<param name="mtIsolate" value="1.5011mm 0.1499mm 0.2007mm 0.1499mm 0.2007mm 0.1499mm 0.2007mm 0.1499mm 0.2007mm 0.1499mm 0.2007mm 0.1499mm 0.2007mm 0.1499mm 0.2007mm"/>
+<param name="mtCopper" value="0.035559375mm 0.0356mm 0.0356mm 0.0356mm 0.0356mm 0.0356mm 0.0356mm 0.0356mm 0.0356mm 0.0356mm 0.0356mm 0.0356mm 0.0356mm 0.0356mm 0.0356mm 0.035559375mm"/>
+<param name="mtIsolate" value="1.6mm 0.1499mm 0.2007mm 0.1499mm 0.2007mm 0.1499mm 0.2007mm 0.1499mm 0.2007mm 0.1499mm 0.2007mm 0.1499mm 0.2007mm 0.1499mm 0.2007mm"/>
 <param name="mdWireWire" value="6mil"/>
 <param name="mdWirePad" value="6mil"/>
@@
 <param name="mdSmdStop" value="0mil"/>
 <param name="msWidth" value="6mil"/>
-<param name="msDrill" value="13mil"/>
-<param name="msMicroVia" value="13mil"/>
+<param name="msDrill" value="10mil"/>
+<param name="msMicroVia" value="10mil"/>
 <param name="msBlindViaRatio" value="0.5"/>
 <param name="rvPadTop" value="0.25"/>
@@
 <param name="rvMicroViaOuter" value="0.25"/>
 <param name="rvMicroViaInner" value="0.25"/>
-<param name="rlMinPadTop" value="7mil"/>
+<param name="rlMinPadTop" value="5mil"/>
 <param name="rlMaxPadTop" value="20mil"/>
-<param name="rlMinPadInner" value="7mil"/>
+<param name="rlMinPadInner" value="5mil"/>
 <param name="rlMaxPadInner" value="20mil"/>
-<param name="rlMinPadBottom" value="7mil"/>
+<param name="rlMinPadBottom" value="5mil"/>
 <param name="rlMaxPadBottom" value="20mil"/>
-<param name="rlMinViaOuter" value="7mil"/>
+<param name="rlMinViaOuter" value="5mil"/>
 <param name="rlMaxViaOuter" value="20mil"/>
-<param name="rlMinViaInner" value="7mil"/>
+<param name="rlMinViaInner" value="5mil"/>
 <param name="rlMaxViaInner" value="20mil"/>
-<param name="rlMinMicroViaOuter" value="4mil"/>
+<param name="rlMinMicroViaOuter" value="5mil"/>
 <param name="rlMaxMicroViaOuter" value="20mil"/>
-<param name="rlMinMicroViaInner" value="4mil"/>
+<param name="rlMinMicroViaInner" value="5mil"/>
 <param name="rlMaxMicroViaInner" value="20mil"/>
 <param name="psTop" value="-1"/>
@@
 <attribute name="VALUE" x="11.43" y="27.305" size="0.6096" layer="27" rot="R90"/>
 </element>
-<element name="R6" library="resistor" package="R0805" value="10K" x="8.89" y="24.13" smashed="yes" rot="R180">
-<attribute name="NAME" x="9.525" y="22.86" size="0.6096" layer="25" rot="R180"/>
-<attribute name="VALUE" x="9.525" y="26.67" size="0.6096" layer="27" rot="R180"/>
+<element name="R6" library="resistor" package="R0805" value="10K" x="6.985" y="23.495" smashed="yes" rot="R180">
+<attribute name="NAME" x="7.62" y="22.225" size="0.6096" layer="25" rot="R180"/>
+<attribute name="VALUE" x="7.62" y="26.035" size="0.6096" layer="27" rot="R180"/>
 </element>
 <element name="U1" library="Atmel_By_element14_Batch_1-00" package="SOIC127P798X216-8N" value="ATTINY85-20SU" x="16.51" y="22.86" smashed="yes">
@@
 <wire x1="11.43" y1="15.56" x2="21.59" y2="15.56" width="0.8128" layer="1"/>
 <wire x1="3.81" y1="12.7" x2="3.81" y2="13.97" width="0.8128" layer="16"/>
-<via x="5.08" y="16.51" extent="1-16" drill="0.3302"/>
 <via x="29.21" y="16.51" extent="1-16" drill="0.3302"/>
-<wire x1="3.81" y1="21.59" x2="3.81" y2="16.51" width="0.8128" layer="16"/>
-<wire x1="3.81" y1="16.51" x2="3.81" y2="12.7" width="0.8128" layer="16"/>
 <wire x1="8.89" y1="6.03" x2="8.89" y2="12.7" width="0.8128" layer="1"/>
 <wire x1="8.89" y1="12.7" x2="7.62" y2="15.24" width="0.8128" layer="1"/>
@@
 <wire x1="21.59" y1="15.56" x2="21.59" y2="10.48" width="0.8128" layer="1"/>
 <wire x1="21.59" y1="10.48" x2="20.32" y2="9.21" width="0.8128" layer="1"/>
-<wire x1="8.89" y1="26.99" x2="8.89" y2="26.67" width="0.8128" layer="1"/>
-<wire x1="8.89" y1="26.67" x2="7.94" y2="25.72" width="0.8128" layer="1"/>
-<wire x1="7.94" y1="25.72" x2="7.94" y2="24.13" width="0.8128" layer="1"/>
 <wire x1="23.495" y1="23.815" x2="23.18" y2="24.13" width="0.8128" layer="1"/>
 <wire x1="23.18" y1="24.13" x2="22.545" y2="24.765" width="0.8128" layer="1"/>
@@
 <wire x1="7.3" y1="15.56" x2="7.62" y2="15.56" width="0.8128" layer="1"/>
 <wire x1="29.21" y1="12.7" x2="29.21" y2="16.51" width="0.8128" layer="16"/>
-<wire x1="5.08" y1="16.51" x2="3.81" y2="16.51" width="0.8128" layer="16"/>
-<wire x1="3.81" y1="21.59" x2="6.35" y2="24.13" width="0.8128" layer="16"/>
-<via x="6.35" y="24.13" extent="1-16" drill="0.3302"/>
-<wire x1="6.35" y1="24.13" x2="7.94" y2="24.13" width="0.8128" layer="1"/>
-<wire x1="5.08" y1="16.51" x2="6.03" y2="15.56" width="0.8128" layer="1"/>
-<wire x1="6.03" y1="15.56" x2="7.62" y2="15.56" width="0.8128" layer="1"/>
 <wire x1="29.21" y1="16.51" x2="28.26" y2="15.56" width="0.8128" layer="1"/>
 <wire x1="28.26" y1="15.56" x2="25.4" y2="15.56" width="0.8128" layer="1"/>
+<wire x1="8.89" y1="26.99" x2="7.3" y2="25.4" width="0.8128" layer="1"/>
+<wire x1="7.3" y1="25.4" x2="6.35" y2="25.4" width="0.8128" layer="1"/>
+<wire x1="6.35" y1="25.4" x2="6.035" y2="25.085" width="0.8128" layer="1"/>
+<wire x1="6.035" y1="25.085" x2="6.035" y2="23.495" width="0.8128" layer="1"/>
+<wire x1="6.035" y1="23.495" x2="5.08" y2="22.54" width="0.8128" layer="1"/>
+<wire x1="5.08" y1="22.54" x2="5.08" y2="16.51" width="0.8128" layer="1"/>
+<via x="5.08" y="16.51" extent="1-16" drill="0.6"/>
+<wire x1="5.08" y1="16.51" x2="3.81" y2="15.24" width="0.8128" layer="16"/>
+<wire x1="3.81" y1="15.24" x2="3.81" y2="12.7" width="0.8128" layer="16"/>
+<wire x1="7.62" y1="15.56" x2="6.03" y2="15.56" width="0.8128" layer="1"/>
+<wire x1="6.03" y1="15.56" x2="5.08" y2="16.51" width="0.8128" layer="1"/>
 <wire x1="7.62" y1="15.24" x2="7.62" y2="15.56" width="0" layer="19" extent="1-1"/>
 </signal>
@@
 <contactref element="U1" pad="2"/>
 <contactref element="LED1" pad="4-DIN"/>
-<wire x1="12.8016" y1="23.495" x2="12.065" y2="23.495" width="0.8128" layer="1"/>
-<wire x1="12.065" y1="23.495" x2="10.16" y2="21.59" width="0.8128" layer="1"/>
-<wire x1="10.16" y1="21.59" x2="6.35" y2="21.59" width="0.8128" layer="1"/>
-<wire x1="6.35" y1="21.59" x2="5.08" y2="22.86" width="0.8128" layer="1"/>
-<wire x1="5.08" y1="22.86" x2="5.08" y2="26.38" width="0.8128" layer="1"/>
-<wire x1="5.08" y1="26.38" x2="5.46" y2="26.76" width="0.8128" layer="1"/>
+<wire x1="12.8016" y1="23.495" x2="10.795" y2="23.495" width="0.8128" layer="1"/>
+<wire x1="10.795" y1="23.495" x2="10.16" y2="22.86" width="0.8128" layer="1"/>
+<via x="10.16" y="22.86" extent="1-16" drill="0.6"/>
+<wire x1="10.16" y1="22.86" x2="5.08" y2="22.86" width="0.8128" layer="16"/>
+<wire x1="5.08" y1="22.86" x2="3.81" y2="24.13" width="0.8128" layer="16"/>
+<via x="3.81" y="24.13" extent="1-16" drill="0.6"/>
+<wire x1="3.81" y1="24.13" x2="3.81" y2="25.11" width="0.8128" layer="1"/>
+<wire x1="3.81" y1="25.11" x2="5.46" y2="26.76" width="0.8128" layer="1"/>
 </signal>
 <signal name="RESET">
@@
 <contactref element="U1" pad="1"/>
 <contactref element="J1" pad="4"/>
-<wire x1="9.84" y1="24.13" x2="10.475" y2="24.765" width="0.8128" layer="1"/>
-<wire x1="10.475" y1="24.765" x2="12.8016" y2="24.765" width="0.8128" layer="1"/>
 <wire x1="12.8016" y1="24.765" x2="12.8016" y2="26.7716" width="0.8128" layer="1"/>
 <wire x1="12.8016" y1="26.7716" x2="13.97" y2="27.94" width="0.8128" layer="1"/>
@@
 <via x="17.78" y="27.94" extent="1-16" drill="0.3302"/>
 <wire x1="17.78" y1="27.94" x2="17.78" y2="30.095" width="0.8128" layer="16"/>
+<wire x1="12.8016" y1="24.765" x2="9.205" y2="24.765" width="0.8128" layer="1"/>
+<wire x1="9.205" y1="24.765" x2="7.935" y2="23.495" width="0.8128" layer="1"/>
 </signal>
 <signal name="TEMP">
@@
 <via x="10.16" y="10.16" extent="1-16" drill="0.3302"/>
 <via x="10.16" y="20.32" extent="1-16" drill="0.3302"/>
+<wire x1="10.16" y1="20.32" x2="10.16" y2="10.16" width="0.8128" layer="16"/>
 <wire x1="12.8016" y1="22.225" x2="12.065" y2="22.225" width="0.8128" layer="1"/>
 <wire x1="12.065" y1="22.225" x2="10.16" y2="20.32" width="0.8128" layer="1"/>
-<wire x1="10.16" y1="20.32" x2="10.16" y2="10.16" width="0.8128" layer="16"/>
 </signal>
 <signal name="MOSI/SDA">

Commit message: minor fixes
Routing:
- net N$7: track 3.12 -> 26.4 mm
- net VCC: track 87.8 -> 89.6 mm

Commit message: Cleaned up for entry
Parts:
- added FRAME1: FRAME-LETTER, SparkFun-Aesthetics:CREATIVE_COMMONS
Changed lines of the file:
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@@
 </element>
 <element name="LOGO1" library="SparkFun-Aesthetics" package="OSHW-LOGO-L" value="OSHW-LOGOL" x="16.51" y="4.445" smashed="yes"/>
+<element name="FRAME1" library="SparkFun-Aesthetics" package="CREATIVE_COMMONS" value="FRAME-LETTER" x="17" y="-14"/>
 </elements>
 <signals>
